Commit message: revised files so that they can work in ROS Hydro and gazebo 1.9

File: swivel_description/model/swivel_test.urdf.xacro (robot description, xacro)
@@ -5,5 +5,5 @@
   <!-- ros_control plugin -->
    <gazebo>
-      <plugin name="ros_control" filename="libros_control_gazebo_plugin.so">
+      <plugin name="gazebo_ros_control" filename="libros_control_gazebo_plugin.so">
         <ns>/swivel</ns>
       </plugin>
@@ -13,5 +13,5 @@
       <origin xyz="0 0 0" rpy="0 0 0" />
       <geometry >
-	<mesh filename="package://swivel_description/meshes/Swivel_Base.STL" />
+	<mesh filename="package://swivel_description/meshes/Swivel_Base.stl" />
       </geometry>
       <material name="SwivelLightGray" />
@@ -26,5 +26,5 @@
       <origin xyz="0 0 0.06" rpy="0 0 0" />
       <geometry >
-	<mesh filename="package://swivel_description/meshes/Swivel_Link_1.STL" />
+	<mesh filename="package://swivel_description/meshes/Swivel_Link_1.stl" />
       </geometry>
       <material name="SwivelLightGray" />
@@ -48,5 +48,5 @@
       <origin xyz="0 0 0" rpy="0 0 0" />
       <geometry >
-	<mesh filename="package://swivel_description/meshes/Swivel_Link_2.STL" />
+	<mesh filename="package://swivel_description/meshes/Swivel_Link_2.stl" />
       </geometry>
       <material name="SwivelRed" />
